Commit message: Raised the stands so that they are visible to the lidar. Moved the kinect so that it can see the cubes

File: manipulation/ws_husky_abb/husky_custom_description/urdf/custom_description.urdf.xacro (robot description, xacro)
@@ -44,5 +44,5 @@
   </joint>
   <joint name="kinect_frame_joint" type="fixed">
-    <origin xyz="0.32 0 -0.05" rpy="0 0 0"/>
+    <origin xyz="0.39 -0.25 .042" rpy=".032 0 0.4051"/>
     <parent link="top_plate_link"/>
     <child link="camera_link"/>
