Commit message: replaced kinect with d435

File: mobile_manipulation/ws_husky_abb/husky_abb_description/urdf/husky_abb.urdf.xacro (robot description, xacro)
@@ -5,5 +5,5 @@
   <xacro:include filename="$(find husky_description)/urdf/husky.urdf.xacro"/>
   <xacro:include filename="$(find barrett_hand)/urdf/barrett.xacro"/>
-  <xacro:include filename="$(find husky_abb_description)/urdf/kinect.xacro"/>
+  <!-- <xacro:include filename="$(find husky_abb_description)/urdf/kinect.xacro"/> -->
   <!-- Fix robot to Gazebo world
   <link name="world"/>-->

File: mobile_manipulation/ws_husky_abb/husky_custom_description/urdf/custom_description.urdf.xacro (robot description, xacro)
@@ -31,4 +31,5 @@
   <xacro:include filename="$(find husky_description)/urdf/accessories/intel_realsense.urdf.xacro"/>
 <!--END of mobility+manipulation includes-->
+<link name="camera_link"/>
   <joint name="husky_abb" type="fixed">
   	<origin xyz="0.3 0 0.253" rpy="0 0 0"/>
@@ -43,9 +44,9 @@
     <child link="barrett_base_link"/>
   </joint>
-  <joint name="kinect_frame_joint" type="fixed">
+  <joint name="realsense_frame_joint" type="fixed">
     <origin xyz="0.39 -0.25 .042" rpy=".032 0 0.4051"/>
     <parent link="top_plate_link"/>
     <child link="camera_link"/>
   </joint>
-  <xacro:intel_realsense_mount prefix="camera" topic="test" parent_link="base_link"/>
+  <xacro:intel_realsense_mount prefix="camera" topic="realsense" parent_link="camera_link"/>
 </robot>
